File: PCB/UPZ_Switcher/IO.sch (KiCad schematic (older format))
At the start: 108 parts, among them Q1 BS170F, Q10 BS170F, Q11 BS170F, Q12 BS170F, Q13 BS170F, Q14 BS170F, Q15 BS170F, Q16 BS170F, Q17 BS170F, Q18 BS170F, Q2 BS170F, Q3 BS170F, Q4 BS170F, Q5 BS170F, Q6 BS170F, Q7 BS170F, Q8 BS170F, Q9 BS170F, U1 MCP23017_SP, U2 MCP23017_SP, U3 MCP23017_SP

Commit message: Started PCB design
Parts:
- added C19, C20: 10nF, Capacitor_SMD:C_1206_3216Metric, symbol Device:C_Small
- added D19, D20: 1N4148W, Diode_SMD:D_SOD-123, symbol Diode:1N4148W
- added Q19, Q20: BS170F, Package_TO_SOT_SMD:SOT-23, symbol Transistor_FET:BS170F
- added R42, R43: 1K, Resistor_SMD:R_1206_3216Metric, symbol Device:R_Small_US
- C2: footprint (none) -> Capacitor_SMD:C_1206_3216Metric
- U1, U2, U3: footprint Package_DIP:DIP-28_W7.62mm -> Package_SO:SOIC-28W_7.5x17.9mm_P1.27mm
Connections:
- net GND: now also C19.2, C20.2, Q19.2 (S), Q20.2 (S)
- net at U2.3 (GPB2): now also R42.2
- net at U2.4 (GPB3): now also R43.2
- net 5V_Relay renamed K1+
- net K1+: now also D19.1 (K), D20.1 (K)
- new net: C20.1, Q20.1 (G), R43.1
- new net: C19.1, Q19.1 (G), R42.1
- new net K19-: D19.2 (A), Q19.3 (D)
- new net K20-: D20.2 (A), Q20.3 (D)
Other:
- moved on the sheet: C13, C18, D11, D12, D13, D14, D15, D16, D17, D18, LED10, LED9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

Commit message: Relay Board finished
Parts:
- U1, U2, U3: footprint Package_SO:SOIC-28W_7.5x17.9mm_P1.27mm -> Package_DIP:DIP-28_W7.62mm_Socket_LongPads
Connections:
- net VDD is gone; now on net K1+: R39.2, R44.2, R45.2, U1.9 (VDD), U2.15 (A0), U2.9 (VDD), U3.16 (A1), U3.9 (VDD)
- net MCP3.4: now reaches U2.4 (GPB3)
- net MCP3.4: now also R26.2; no longer R43.2
- net MCP2.1: now reaches R42.2
- net MCP2.1: now also U3.1 (GPB0); no longer U2.3 (GPB2)
- net MCP1.1: now reaches R1.2, U1.1 (GPB0)
- net MCP1.2: now reaches U1.2 (GPB1)
- net MCP1.2: now also R9.2; no longer R2.2
- net MCP1.9: now reaches U1.21 (GPA0)
- net MCP1.9: now also R3.2; no longer R9.2
- net MCP1.10: now reaches U1.22 (GPA1)
- net MCP1.10: now also R11.2; no longer R10.2
- net MCP1.11: now reaches U1.23 (GPA2)
- net MCP1.11: now also R35.2; no longer R11.2
- net MCP1.12: now reaches U1.24 (GPA3)
- net MCP1.12: now also R36.2; no longer R12.2
- net MCP1.13: now reaches U1.25 (GPA4)
- net MCP1.13: now also R4.2; no longer R13.2
- net MCP1.14: now reaches U1.26 (GPA5)
- net MCP1.14: now also R12.2; no longer R14.2
- net MCP1.15: now reaches U1.27 (GPA6)
- net MCP1.15: now also R27.2; no longer R15.2
- net MCP1.16: now reaches U1.28 (GPA7)
- net MCP1.16: now also R28.2; no longer R16.2
- net MCP1.3: now reaches U1.3 (GPB2)
- net MCP1.3: now also R37.2; no longer R3.2
- net MCP1.4: now reaches U1.4 (GPB3)
- net MCP1.4: now also R38.2; no longer R4.2
- net MCP1.5: now reaches U1.5 (GPB4)
- net MCP1.5: now also R2.2; no longer R5.2
- net MCP1.6: now reaches U1.6 (GPB5)
- net MCP1.6: now also R10.2; no longer R6.2
- net MCP1.7: now reaches U1.7 (GPB6)
- net MCP1.7: now also R33.2; no longer R7.2
- net MCP1.8: now reaches U1.8 (GPB7)
- net MCP1.8: now also R34.2; no longer R8.2
- net MCP2.2: now reaches R17.2
- net MCP2.2: now also U3.2 (GPB1); no longer U2.1 (GPB0)
- net MCP3.2: now reaches U2.2 (GPB1)
- net MCP3.2: now also R16.2; no longer R18.2
- net MCP3.9: now reaches U2.21 (GPA0)
- net MCP3.10: now reaches U2.22 (GPA1)
- net MCP3.11: now reaches U2.23 (GPA2)
- net MCP3.12: now reaches U2.24 (GPA3)
- net MCP2.3: now reaches R19.2
- net MCP2.3: now also U3.3 (GPB2); no longer U2.25 (GPA4)
- net MCP2.4: now reaches R20.1
- net MCP2.4: now also U3.4 (GPB3); no longer U2.26 (GPA5)
- net MCP3.15: now reaches U2.27 (GPA6)
- net MCP3.15: no longer R21.2
- net MCP3.16: now reaches U2.28 (GPA7)
- net MCP3.16: no longer R22.1
- net MCP3.5: now reaches U2.5 (GPB4)
- net MCP3.5: now also R43.2
- net MCP3.6: now reaches U2.6 (GPB5)
- net MCP3.6: now also R18.2
- net MCP3.7: now reaches U2.7 (GPB6)
- net MCP3.7: now also R21.2
- net MCP3.8: now reaches U2.8 (GPB7)
- net MCP3.8: now also R22.1
- net MCP2.15: now reaches R23.2
- net MCP2.15: now also U3.27 (GPA6); no longer U3.1 (GPB0)
- net MCP2.16: now reaches R24.2
- net MCP2.16: now also U3.28 (GPA7); no longer U3.2 (GPB1)
- net MCP2.11: now reaches R31.2
- net MCP2.11: now also U3.23 (GPA2); no longer U3.21 (GPA0)
- net MCP2.10: now reaches U3.22 (GPA1)
- net MCP2.10: now also R14.2; no longer R32.2
- net MCP2.12: now reaches U3.24 (GPA3)
- net MCP2.12: now also R32.2; no longer R34.2
- net MCP2.13: now reaches U3.25 (GPA4)
- net MCP2.13: now also R7.2; no longer R35.2
- net MCP2.14: now reaches U3.26 (GPA5)
- net MCP2.14: now also R15.2; no longer R36.2
- net MCP3.3: now reaches R25.2
- net MCP3.3: now also U2.3 (GPB2); no longer U3.3 (GPB2)
- net MCP2.5: now reaches U3.5 (GPB4)
- net MCP2.5: now also R5.2; no longer R27.2
- net MCP2.6: now reaches U3.6 (GPB5)
- net MCP2.6: now also R13.2; no longer R28.2
- net MCP2.7: now reaches R29.2, U3.7 (GPB6)
- net MCP2.8: now reaches R30.2, U3.8 (GPB7)
- new net MCP2.9: R6.2, U3.21 (GPA0)
- new net MCP3.1: R8.2, U2.1 (GPB0)
- new net MCP3.13: U2.25 (GPA4)
- new net MCP3.14: U2.26 (GPA5)
Other:
- moved on the sheet: D1, D10, D11, D12, D13, D14, D15, D16, D17, D18, D19, D2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
