File: PCB/UPZ_Switcher/Power Supply.sch (KiCad schematic (older format))
At the start: 0 parts

Commit message: Updated schematic, PSU added + draft program
Parts:
- added C? (x2): 4700uF, symbol Device:CP
- added C?: 100uF, symbol Device:CP
- added C? (x7): 100nF, symbol Device:C
- added C?: 1000uF, symbol Device:CP
- added C?: 220nF, symbol Device:C
- added D? (x3): 1N5408, Diode_THT:D_DO-201AD_P15.24mm_Horizontal, symbol Diode:1N5408
- added D? (x6): 1N4007, Diode_THT:D_DO-41_SOD81_P10.16mm_Horizontal, symbol Diode:1N4007
- added D?: D_Bridge_+-AA, symbol Device:D_Bridge_+-AA
- added F? (x2): Fuse, symbol Device:Fuse
- added IC?: TL783CKCSE3, TO254P470X1016X1965-3P, symbol BVKSound:TL783CKCSE3
- added P?: Conn_WallPlug_Earth, symbol Connector:Conn_WallPlug_Earth
- added R?: 150R, symbol Device:R_Small
- added R? (x4): 6K8, symbol Device:R_Small
- added R?: 47R, symbol Device:R_Small
- added RV?: 5K6, symbol Device:R_POT_TRIM
- added TR? (x2): TRANSF1, symbol Transformer:TRANSF1
- added U? (x2): PR2301_TruePhantom, Package_SO:SO-8_3.9x4.9mm_P1.27mm, symbol BVKSound:PR2301_TruePhantom
- added U?: L7805, symbol Regulator_Linear:L7805
Connections:
- net labels added: 5V, 5V_Gnd, GND, GND1, Phantom_48V_COLD_A, Phantom_48V_COLD_B, Phantom_48V_HOT_A, Phantom_48V_HOT_B, Phantom_GND
- wire segments 0 -> 144

Commit message: Started PCB design
Parts:
- gave numbers to parts that had none: 38

Commit message: updated phantom design + MCU board
Parts:
- removed C11, C12: 100nF, symbol Device:C
- removed D10, D7, D8, D9: 1N4007, Diode_THT:D_DO-41_SOD81_P10.16mm_Horizontal, symbol Diode:1N4007
- removed R2: 47R, symbol Device:R_Small
- removed R3, R4, R5, R6: 6K8, symbol Device:R_Small
- removed RV1: 5K6, symbol Device:R_POT_TRIM
- removed U2, U3: PR2301_TruePhantom, Package_SO:SO-8_3.9x4.9mm_P1.27mm, symbol BVKSound:PR2301_TruePhantom
- added R?: 5K6, symbol Device:R_Small
Connections:
- net labels added: 5V_GND, Phantom_48V, Phantom_48V_GND
- net labels removed: 5V_Gnd, Phantom_48V_COLD_A, Phantom_48V_COLD_B, Phantom_48V_HOT_A, Phantom_48V_HOT_B, Phantom_GND
- wire segments 144 -> 97

Commit message: update on power supply
Parts:
- removed C1, C2, C7, C8, C9: 100nF, symbol Device:C
- removed C10: 100uF, symbol Device:CP
- removed C3: 220nF, symbol Device:C
- removed C5: 4700uF, symbol Device:CP
- removed C6: 1000uF, symbol Device:CP
- removed D1, D2, D6: 1N5408, Diode_THT:D_DO-201AD_P15.24mm_Horizontal, symbol Diode:1N5408
- removed D3: D_Bridge_+-AA, symbol Device:D_Bridge_+-AA
- removed D4, D5: 1N4007, Diode_THT:D_DO-41_SOD81_P10.16mm_Horizontal, symbol Diode:1N4007
- removed F1, F2: Fuse, symbol Device:Fuse
- removed IC1: TL783CKCSE3, TO254P470X1016X1965-3P, symbol BVKSound:TL783CKCSE3
- removed P1: Conn_WallPlug_Earth, symbol Connector:Conn_WallPlug_Earth
- removed R1: 150R, symbol Device:R_Small
- removed R?: 5K6, symbol Device:R_Small
- removed TR1, TR2: TRANSF1, symbol Transformer:TRANSF1
- removed U1: L7805, symbol Regulator_Linear:L7805
- added C1, C2: 100nF, Capacitor_SMD:C_1206_3216Metric, symbol Device:C_Small
- added C3: 100uF, Capacitor_THT:CP_Radial_D10.0mm_P5.00mm, symbol Device:CP
- added J1, J2: 1-726386-2, 17263862, symbol BVKSound:1-726386-2
- added J3: 71918-110LF, BVKSound:71918-110LF, symbol BVKSound:71918-110LF
- added U1: MP-LD05-23B05R2, BVKSound:MP-LD05-23B05R2, symbol BVKSound:MP-LD05-23B05R2
- added U2: VCE05US48, BVKSound:VCE05US48, symbol BVKSound:VCE05US48
- C4: value 4700uF -> 100uF; footprint (none) -> Capacitor_THT:CP_Radial_D10.0mm_P5.00mm
Connections:
- net labels removed: GND, GND1
- wire segments 97 -> 57
