File: PCB/UPZ_Switcher/Relay.sch (KiCad schematic (older format))
At the start: 28 parts, among them K1 TQ2SA-5V-Z, K10 TQ2SA-5V-Z, K11 TQ2SA-5V-Z, K12 TQ2SA-5V-Z, K13 TQ2SA-5V-Z, K14 TQ2SA-5V-Z, K15 TQ2SA-5V-Z, K16 TQ2SA-5V-Z, K17 TQ2SA-5V-Z, K18 TQ2SA-5V-Z, K2 TQ2SA-5V-Z, K3 TQ2SA-5V-Z, K4 TQ2SA-5V-Z, K5 TQ2SA-5V-Z, K6 TQ2SA-5V-Z, K7 TQ2SA-5V-Z, K8 TQ2SA-5V-Z, K9 TQ2SA-5V-Z

Commit message: Started PCB design
Parts:
- added K19, K20: TQ2SA-5V-Z, BVKSound:TQ2SAL23VZ, symbol BVKSound:TQ2SA-5V-Z
Connections:
- net BUSB.G is gone; now on net BUSA.G: BUS_B1.G1
- net BUSBMH is gone; now on net BUSAMH: BUS_B1.MH1
- net IN1.1 is gone; now on net GND2: Input_1.1
- net IN1.4 is gone; now on net BUSAMH: Input_1.4
- net IN1.5 is gone; now on net BUSA.G: Input_1.5
- net IN2.1 is gone; now on net GND2: Input_2.1
- net IN2.4 is gone; now on net BUSAMH: Input_2.4
- net IN2.5 is gone; now on net BUSA.G: Input_2.5
- net IN3.1 is gone; now on net GND2: Input_3.1
- net IN3.4 is gone; now on net BUSAMH: Input_3.4
- net IN3.5 is gone; now on net BUSA.G: Input_3.5
- net IN4.1 is gone; now on net GND2: Input_4.1
- net IN4.4 is gone; now on net BUSAMH: Input_4.4
- net IN4.5 is gone; now on net BUSA.G: Input_4.5
- net IN5.1 is gone; now on net GND2: Input_5.1
- net IN5.4 is gone; now on net BUSAMH: Input_5.4
- net IN5.5 is gone; now on net BUSA.G: Input_5.5
- net IN6.1 is gone; now on net GND2: Input_6.1
- net IN6.4 is gone; now on net BUSAMH: Input_6.4
- net IN6.5 is gone; now on net BUSA.G: Input_6.5
- net IN7.1 is gone; now on net GND2: Input_7.1
- net IN7.4 is gone; now on net BUSAMH: Input_7.4
- net IN7.5 is gone; now on net BUSA.G: Input_7.5
- net IN8.1 is gone; now on net GND2: Input_8.1
- net IN8.4 is gone; now on net BUSAMH: Input_8.4
- net IN8.5 is gone; now on net BUSA.G: Input_8.5
- net BUSA.2: now also K19.4 (N.O._1); no longer BUS_A1.2
- net BUSA.3: now also K19.7 (N.O._2); no longer BUS_A1.3
- net BUSB.2: now also K20.4 (N.O._1); no longer BUS_B1.2
- net BUSB.3: now also K20.7 (N.O._2); no longer BUS_B1.3
- new net K19+: K19.1 (COIL_+)
- new net K19-: K19.10 (COIL_-)
- new net K20+: K20.1 (COIL_+)
- new net K20-: K20.10 (COIL_-)
- new net OUTA.2: BUS_A1.2, K19.3 (COM_1)
- new net OUTA.3: BUS_A1.3, K19.8 (COM_2)
- new net OUTB.2: BUS_B1.2, K20.3 (COM_1)
- new net OUTB.3: BUS_B1.3, K20.8 (COM_2)

Commit message: updated phantom design + MCU board
Parts:
- added C21, C22, C23, C24: 47uF, Capacitor_THT:CP_Radial_D8.0mm_P3.50mm, symbol Device:CP1_Small
- added R44, R45, R46, R47: 6K8, Resistor_SMD:R_1206_3216Metric, symbol Device:R_Small_US
Connections:
- net OUTA.2: now also C22.1; no longer K19.3 (COM_1)
- net OUTA.3: now also C21.1; no longer K19.8 (COM_2)
- net OUTB.2: now also C24.1; no longer K20.3 (COM_1)
- net OUTB.3: now also C23.1; no longer K20.8 (COM_2)
- net Phantom_48V_COLD_A: no longer names the net of K17.8 (COM_2)
- net Phantom_48V_COLD_A: now also R45.2
- net Phantom_48V_COLD_B: no longer names the net of K18.8 (COM_2)
- net Phantom_48V_COLD_B: now also R47.2
- net Phantom_48V_HOT_A: no longer names the net of K17.3 (COM_1)
- net Phantom_48V_HOT_A: now also R44.1
- net Phantom_48V_HOT_B: no longer names the net of K18.3 (COM_1)
- net Phantom_48V_HOT_B: now also R46.1
- new net: C22.2, K19.3 (COM_1)
- new net: C21.2, K19.8 (COM_2)
- new net: C24.2, K20.3 (COM_1)
- new net: C23.2, K20.8 (COM_2)
- new net Phantom_48V: R44.2, R45.1, R46.2, R47.1
Other:
- moved on the sheet: K19, K20

Commit message: final
Connections:
- net BUSA.2: now also K1.8 (COM_2), K17.7 (N.O._2), K19.7 (N.O._2), K2.8 (COM_2), K3.8 (COM_2), K4.8 (COM_2), K5.8 (COM_2), K6.8 (COM_2), K7.8 (COM_2), K8.8 (COM_2); no longer K1.3 (COM_1), K17.4 (N.O._1), K19.4 (N.O._1), K2.3 (COM_1), K3.3 (COM_1), K4.3 (COM_1), K5.3 (COM_1), K6.3 (COM_1), K7.3 (COM_1), K8.3 (COM_1)
- net BUSA.3: now also K1.3 (COM_1), K17.4 (N.O._1), K19.4 (N.O._1), K2.3 (COM_1), K3.3 (COM_1), K4.3 (COM_1), K5.3 (COM_1), K6.3 (COM_1), K7.3 (COM_1), K8.3 (COM_1); no longer K1.8 (COM_2), K17.7 (N.O._2), K19.7 (N.O._2), K2.8 (COM_2), K3.8 (COM_2), K4.8 (COM_2), K5.8 (COM_2), K6.8 (COM_2), K7.8 (COM_2), K8.8 (COM_2)
- net BUSA.G: no longer BUS_B1.G1, Input_1.5, Input_2.5, Input_3.5, Input_4.5, Input_5.5, Input_6.5, Input_7.5, Input_8.5
- net BUSAMH: no longer BUS_B1.MH1, Input_1.4, Input_2.4, Input_3.4, Input_4.4, Input_5.4, Input_6.4, Input_7.4, Input_8.4
- net BUSB.2: now also K10.8 (COM_2), K11.8 (COM_2), K12.8 (COM_2), K13.8 (COM_2), K14.8 (COM_2), K15.8 (COM_2), K16.8 (COM_2), K18.7 (N.O._2), K20.7 (N.O._2), K9.8 (COM_2); no longer K10.3 (COM_1), K11.3 (COM_1), K12.3 (COM_1), K13.3 (COM_1), K14.3 (COM_1), K15.3 (COM_1), K16.3 (COM_1), K18.4 (N.O._1), K20.4 (N.O._1), K9.3 (COM_1)
- net BUSB.3: now also K10.3 (COM_1), K11.3 (COM_1), K12.3 (COM_1), K13.3 (COM_1), K14.3 (COM_1), K15.3 (COM_1), K16.3 (COM_1), K18.4 (N.O._1), K20.4 (N.O._1), K9.3 (COM_1); no longer K10.8 (COM_2), K11.8 (COM_2), K12.8 (COM_2), K13.8 (COM_2), K14.8 (COM_2), K15.8 (COM_2), K16.8 (COM_2), K18.7 (N.O._2), K20.7 (N.O._2), K9.8 (COM_2)
- net IN1.2: now also K1.7 (N.O._2), K9.7 (N.O._2); no longer K1.4 (N.O._1), K9.4 (N.O._1)
- net IN1.3: now also K1.4 (N.O._1), K9.4 (N.O._1); no longer K1.7 (N.O._2), K9.7 (N.O._2)
- net IN2.2: now also K10.7 (N.O._2), K2.7 (N.O._2); no longer K10.4 (N.O._1), K2.4 (N.O._1)
- net IN2.3: now also K10.4 (N.O._1), K2.4 (N.O._1); no longer K10.7 (N.O._2), K2.7 (N.O._2)
- net IN3.2: now also K11.7 (N.O._2), K3.7 (N.O._2); no longer K11.4 (N.O._1), K3.4 (N.O._1)
- net IN3.3: now also K11.4 (N.O._1), K3.4 (N.O._1); no longer K11.7 (N.O._2), K3.7 (N.O._2)
- net IN4.2: now also K12.7 (N.O._2), K4.7 (N.O._2); no longer K12.4 (N.O._1), K4.4 (N.O._1)
- net IN4.3: now also K12.4 (N.O._1), K4.4 (N.O._1); no longer K12.7 (N.O._2), K4.7 (N.O._2)
- net IN5.2: now also K13.7 (N.O._2), K5.7 (N.O._2); no longer K13.4 (N.O._1), K5.4 (N.O._1)
- net IN5.3: now also K13.4 (N.O._1), K5.4 (N.O._1); no longer K13.7 (N.O._2), K5.7 (N.O._2)
- net IN6.2: now also K14.7 (N.O._2), K6.7 (N.O._2); no longer K14.4 (N.O._1), K6.4 (N.O._1)
- net IN6.3: now also K14.4 (N.O._1), K6.4 (N.O._1); no longer K14.7 (N.O._2), K6.7 (N.O._2)
- net IN7.2: now also K15.7 (N.O._2), K7.7 (N.O._2); no longer K15.4 (N.O._1), K7.4 (N.O._1)
- net IN7.3: now also K15.4 (N.O._1), K7.4 (N.O._1); no longer K15.7 (N.O._2), K7.7 (N.O._2)
- net IN8.2: now also K16.7 (N.O._2), K8.7 (N.O._2); no longer K16.4 (N.O._1), K8.4 (N.O._1)
- net IN8.3: now also K16.4 (N.O._1), K8.4 (N.O._1); no longer K16.7 (N.O._2), K8.7 (N.O._2)
- net OUTA.2: now also C21.1; no longer C22.1
- net OUTA.3: now also C22.1; no longer C21.1
- net OUTB.2: now also C23.1; no longer C24.1
- net OUTB.3: now also C24.1; no longer C23.1
- new net BUSB.G: BUS_B1.G1
- new net BUSBMH: BUS_B1.MH1
- new net IN1.4: Input_1.4
- new net IN1.5: Input_1.5
- new net IN2.4: Input_2.4
- new net IN2.5: Input_2.5
- new net IN3.4: Input_3.4
- new net IN3.5: Input_3.5
- new net IN4.4: Input_4.4
- new net IN4.5: Input_4.5
- new net IN5.4: Input_5.4
- new net IN5.5: Input_5.5
- new net IN6.4: Input_6.4
- new net IN6.5: Input_6.5
- new net IN7.4: Input_7.4
- new net IN7.5: Input_7.5
- new net IN8.4: Input_8.4
- new net IN8.5: Input_8.5
